File: board/gas-motor-driver/gas-motor-driver.kicad_sch (KiCad schematic)
At the start: 9 parts, among them J1 Conn_01x03_Socket, J2 Conn_01x02_Socket, J3 Conn_01x03_Socket, K1 Relay_SPST-NO, K2 Relay_SPST-NO, K3 Relay_SPST-NO, U1 ULN2003

Commit message: Бляха. Здається SoftSerial конфліктує з Servo.
Parts:
- added J4, J7: Conn_01x05_Socket, symbol Connector:Conn_01x05_Socket
- added J5: Conn_01x04_Socket, symbol Connector:Conn_01x04_Socket
- added J6: Conn_01x03_Socket, symbol Connector:Conn_01x03_Socket
Connections:
- net GND: now also J5.1 (Pin_1)
- net LED: now reaches A1.16 (D13)
- net LED: no longer J3.1 (Pin_1)
- net SERVO: now reaches A1.12 (D9)
- net SERVO: now also J3.1 (Pin_1)
- net TEL_RX: now reaches A1.13 (D10)
- net TEL_RX: now also J5.4 (Pin_4)
- net ACC: now reaches A1.5 (D2)
- net ACC: now also U1.1 (I1)
- net START: now reaches A1.6 (D3)
- net START: now also U1.2 (I2)
- net DECOMPRESS: now reaches A1.7 (D4)
- net DECOMPRESS: now also U1.3 (I3)
- new net: J4.1 (Pin_1), J7.1 (Pin_1)
- new net: J4.2 (Pin_2), J7.2 (Pin_2)
- new net: J4.3 (Pin_3), J7.3 (Pin_3)
- new net: J4.4 (Pin_4), J7.4 (Pin_4)
- new net: J4.5 (Pin_5), J7.5 (Pin_5)
Other:
- note added: "1-НЕІЗОЛЬОВАНИЙ-ЕКРАН"
- note added: "1-ЧОРНИЙ-GND"
- note added: "3-СИНІЙ-RF-RECEIVE"
- note added: "5-ЖОВТИЙ-+12В"
- note added: "5-ЧЕРВОНИЙ-+5В"
- note added: "Можливо сюди заведемо живлення."
- note added: "Розʼєм на кузові. Круглий, захищений. 2-3 штуки."
- note added: "Розʼєм приймача на старому польотнику."
- note added: "Розʼєми на розмножувачі сигалів. 5 шт"
- moved on the sheet: A1

Commit message: Хочу спати.
Connections:
- net TEL_RX: now also A1.11 (D8), J5.3 (Pin_3); no longer A1.13 (D10), J5.4 (Pin_4)
Changed lines of the file:
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@@
+	(wire
+		(pts
+			(xy 55.88 81.28) (xy 72.39 81.28)
+		)
+		(stroke
+			(width 0)
+			(type default)
+		)
+	)
 	(wire
 		(pts
@@
 	(wire
 		(pts
-			(xy 54.61 83.82) (xy 72.39 83.82)
+			(xy 55.88 83.82) (xy 72.39 83.82)
 		)
 		(stroke
@@
 	(wire
 		(pts
-			(xy 25.4 86.36) (xy 72.39 86.36)
-		)
-		(stroke
-			(width 0)
-			(type default)
-		)
-	)
-	(wire
-		(pts
 			(xy 144.78 81.28) (xy 144.78 82.55)
 		)
@@
 		(pts
 			(xy 82.55 40.64) (xy 82.55 50.8)
+		)
+		(stroke
+			(width 0)
+			(type default)
+		)
+	)
+	(wire
+		(pts
+			(xy 25.4 83.82) (xy 35.56 83.82)
 		)
 		(stroke
@@
 		)
 	)
+	(label "TEL_RX"
+		(at 35.56 83.82 180)
+		(fields_autoplaced yes)
+		(effects
+			(font
+				(size 1.27 1.27)
+			)
+			(justify right bottom)
+		)
+	)
 	(label "LED"
 		(at 58.42 93.98 0)
@@
 	)
 	(label "SERVO"
-		(at 54.61 83.82 0)
+		(at 55.88 83.82 0)
 		(fields_autoplaced yes)
 		(effects
@@
 	)
 	(label "TEL_RX"
-		(at 35.56 86.36 0)
+		(at 55.88 81.28 0)
 		(fields_autoplaced yes)
 		(effects
